Commit message: ros2 gazebo harmonic migration

File: mini_pupper_description/urdf/mini_pupper_2/mini_pupper_description.urdf.xacro (robot description, xacro)
@@ -367,9 +367,4 @@
   </link>
   <link name="Board_connectors_1">
-    <!-- <inertial>
-      <origin xyz="-0.07276303117117414 -0.002323344081837562 -0.0010631239213060653" rpy="0 0 0"/>
-      <mass value="0.004688613655947816"/>
-      <inertia ixx="0.203205e-6" iyy="1.5404404e-5" izz="1.5546403e-5" ixy="-0.625328e-6" iyz="42.901e-9" ixz="0.186346e-9"/>
-    </inertial> -->
     <visual>
       <origin xyz="-0.061334 3.3e-05 -0.026457" rpy="0 0 0"/>
@@ -387,9 +382,4 @@
   </link>
   <link name="Board_connectors_2">
-    <!-- <inertial>
-      <origin xyz="0.008233541174180986 -0.0021383697865476553 -0.00030110978110910874" rpy="0 0 0"/>
-      <mass value="0.0019746031301169403"/>
-      <inertia ixx="0.458183e-6" iyy="3.284548e-6" izz="3.720196e-6" ixy="-79.741e-9" iyz="4.796e-9" ixz="0.123868e-9"/>
-    </inertial> -->
     <visual>
       <origin xyz="0.045346 5e-06 -0.026457" rpy="0 0 0"/>
@@ -729,5 +719,4 @@
   <link name="Shell_Side">
     <inertial>
-      <!-- <origin xyz="-2.7696824994288393e-05 0.0 0.02237056777957029" rpy="0 0 0"/>  -->
       <origin xyz="-0.00003 0.030005 0.022371" rpy="0 0 0"/>
       <mass value="0.0051928835390001775"/>
@@ -1090,11 +1079,13 @@
     <material>Gazebo/FlatBlack</material>
   </gazebo>
+  <!-- Simplified LIDAR sensor for Gazebo Harmony -->
   <gazebo reference="lidar_link">
     <material>Gazebo/FlatBlack</material>
-    <sensor type="ray" name="lidar">
+    <sensor type="gpu_lidar" name="lidar">
       <always_on>true</always_on>
       <update_rate>30</update_rate>
+      <topic>/scan</topic>
+      <visualize>false</visualize>
       <pose>0 0 0 0 0 0</pose>
-      <visualize>false</visualize>
       <ray>
         <scan>
@@ -1103,5 +1094,5 @@
             <resolution>1</resolution>
             <min_angle>0</min_angle>
-            <max_angle>6.28</max_angle>
+            <max_angle>6.283185307179586</max_angle>
           </horizontal>
         </scan>
@@ -1117,23 +1108,7 @@
         </noise>
       </ray>
-      <plugin name="gazebo_ros_lidar_controller" filename="libgazebo_ros_ray_sensor.so">
-        <ros>
-          <remapping>~/out:=/scan</remapping>
-        </ros>
-        <output_type>sensor_msgs/LaserScan</output_type>
-        <frame_name>lidar_link</frame_name>
-      </plugin>
     </sensor>
   </gazebo>
-  <gazebo>
-    <plugin filename="libgazebo_ros_p3d.so" name="p3d_base_controller">
-      <body_name>base_link</body_name>
-      <frame_name>odom</frame_name>
-      <update_rate>10.0</update_rate>
-      <xyz_offset>0 0 0</xyz_offset>
-      <rpy_offset>0 0 0</rpy_offset>
-      <gaussian_noise>0.01</gaussian_noise>
-    </plugin>
-  </gazebo>
+  <!-- Simplified IMU sensor for Gazebo Harmony -->
   <link name="imu_link">
     <inertial>
@@ -1148,16 +1123,11 @@
   </joint>
   <gazebo reference="imu_link">
-    <sensor name="imu_controller" type="imu">
+    <sensor name="imu_sensor" type="imu">
       <always_on>true</always_on>
       <update_rate>50</update_rate>
-      <plugin name="gazebo_ros_imu_sensor" filename="libgazebo_ros_imu_sensor.so">
-          <ros>
-              <namespace>/imu</namespace>
-              <remapping>~/out:=data</remapping>
-          </ros>
-      </plugin>
+      <topic>/imu/data</topic>
     </sensor>
   </gazebo>
-  <!-- Simulated camera mounted to the front body -->
+  <!-- Simplified Camera sensor for Gazebo Harmony -->
   <link name="camera_link">
     <visual>
@@ -1179,9 +1149,10 @@
   </joint>
   <gazebo reference="camera_link">
-    <sensor type="camera" name="sim_camera">
+    <sensor name="camera" type="camera">
       <always_on>true</always_on>
       <update_rate>30.0</update_rate>
+      <topic>/image_raw</topic>
       <visualize>true</visualize>
-      <camera name="camera">
+      <camera>
         <horizontal_fov>1.3962634</horizontal_fov>
         <image>
@@ -1195,15 +1166,8 @@
         </clip>
       </camera>
-      <!-- Gazebo ROS plugin to publish /image_raw -->
-      <plugin name="camera_controller" filename="libgazebo_ros_camera.so">
-        <always_on>true</always_on>
-        <update_rate>30.0</update_rate>
-        <frame_name>camera_link</frame_name>
-        <image_topic_name>/image_raw</image_topic_name>
-        <!-- camera_info omitted to disable /camera_info -->
-      </plugin>
     </sensor>
   </gazebo>
-  <xacro:mini_pupper_ros2_control use_gazebo_hardware="$(arg use_gazebo_hardware)" />
+  <xacro:mini_pupper_ros2_control use_gazebo_hardware="$(arg use_gazebo_hardware)">
+  </xacro:mini_pupper_ros2_control>
   <!-- Conditional debug support stand -->
   <xacro:if value="$(arg use_debug_stand)">

File: mini_pupper_description/urdf/ros2_control/mini_pupper.ros2_control.xacro (robot description, xacro)
@@ -3,16 +3,5 @@
   <xacro:macro name="pupper_joint" params="joint_name initial_value use_gazebo_hardware">
     <joint name="${joint_name}">
-      <xacro:if value="${use_gazebo_hardware}">
-        <command_interface name="position_pid"/>
-        <!-- Gains tuned for sim_inertia_scale=100 (links are 100x heavier inertially).
-             Joint effective I (hip+distal) ~1.3e-4 kg*m^2, knee ~4.8e-5 kg*m^2.
-             Stability constraint: kd &lt; 2*I/dt_physics ~0.096 (use 0.05 with margin).
-             kp=5.0 gives ~22 ms settling vs 200 ms at kp=1 (within 1-2 gait ticks). -->
-        <param name="pos_kp">5.0</param>
-        <param name="pos_kd">0.05</param>
-      </xacro:if>
-      <xacro:unless value="${use_gazebo_hardware}">
-        <command_interface name="position"/>
-      </xacro:unless>
+      <command_interface name="position"/>
       <state_interface name="position">
         <param name="initial_value">${initial_value}</param>
@@ -24,5 +13,5 @@
     <xacro:if value="${use_gazebo_hardware}">
       <gazebo>
-        <plugin name="gazebo_ros2_control" filename="libgazebo_ros2_control.so">
+          <plugin filename="gz_ros2_control-system" name="gz_ros2_control::GazeboSimROS2ControlPlugin">
           <parameters>$(find mini_pupper_simulation)/config/ros2_control/mini_pupper_2_controllers_sim.yaml</parameters>
           <hold_joints>false</hold_joints>
@@ -33,6 +22,5 @@
       <hardware>
         <xacro:if value="${use_gazebo_hardware}">
-          <plugin>gazebo_ros2_control/GazeboSystem</plugin>
-          <param name="hold_joints">true</param>
+            <plugin>gz_ros2_control/GazeboSimSystem</plugin>
         </xacro:if>
         <xacro:unless value="${use_gazebo_hardware}">

Commit message: Gazebo Harmony - Fixed

File: mini_pupper_description/urdf/mini_pupper_2/mini_pupper_description.urdf.xacro (robot description, xacro)
@@ -36,4 +36,17 @@
     <xacro:property name="sim_inertia_scale" value="100" />
     <xacro:property name="sim_body_inertia_scale" value="100" />
+    <xacro:property name="sim_mass_scale" value="30.0" />
+    <xacro:property name="base_link_mass" value="${0.174884 * sim_mass_scale}" />
+    <xacro:property name="lnkgrp1_mass" value="${0.020769 * sim_mass_scale}" />
+    <xacro:property name="lnkgrp2_mass" value="${0.001906 * sim_mass_scale}" />
+    <xacro:property name="lnkgrp3_mass" value="${0.001144 * sim_mass_scale}" />
+    <xacro:property name="pltgrp1_mass" value="${0.002574 * sim_mass_scale}" />
+    <xacro:property name="pltgrp2_mass" value="${0.002231 * sim_mass_scale}" />
+    <xacro:property name="feet_mass" value="${0.001405 * sim_mass_scale}" />
+    <xacro:property name="body_front_mass" value="${0.00785515871148119 * sim_mass_scale}" />
+    <xacro:property name="board_pcb_mass" value="${0.014261552601793053 * sim_mass_scale}" />
+    <xacro:property name="lidar_mass" value="${0.108 * sim_mass_scale}" />
+    <xacro:property name="shell_side_mass" value="${0.0051928835390001775 * sim_mass_scale}" />
+    <xacro:property name="imu_mass" value="${0.0001 * sim_mass_scale}" />
   </xacro:if>
   <xacro:unless value="$(arg use_gazebo_hardware)">
@@ -42,4 +55,16 @@
     <xacro:property name="sim_inertia_scale" value="1" />
     <xacro:property name="sim_body_inertia_scale" value="1" />
+    <xacro:property name="base_link_mass" value="0.174884" />
+    <xacro:property name="lnkgrp1_mass" value="0.020769" />
+    <xacro:property name="lnkgrp2_mass" value="0.001906" />
+    <xacro:property name="lnkgrp3_mass" value="0.001144" />
+    <xacro:property name="pltgrp1_mass" value="0.002574" />
+    <xacro:property name="pltgrp2_mass" value="0.002231" />
+    <xacro:property name="feet_mass" value="0.001405" />
+    <xacro:property name="body_front_mass" value="0.00785515871148119" />
+    <xacro:property name="board_pcb_mass" value="0.014261552601793053" />
+    <xacro:property name="lidar_mass" value="0.108" />
+    <xacro:property name="shell_side_mass" value="0.0051928835390001775" />
+    <xacro:property name="imu_mass" value="0.0001" />
   </xacro:unless>
   <!-- Link group 1 - lf1, rf1, lb1, rb1 -->
@@ -62,5 +87,5 @@
     <inertial>
       <origin xyz="-0.008867 0.000396 -0.007154" rpy="0 0 0"/>
-      <mass value="0.174884"/>
+      <mass value="${base_link_mass}"/>
       <inertia ixx="${0.00090939 * sim_body_inertia_scale}" iyy="${0.00426716 * sim_body_inertia_scale}" izz="${0.00440707 * sim_body_inertia_scale}" ixy="${1.27324e-7 * sim_body_inertia_scale}" iyz="${1.05509e-9 * sim_body_inertia_scale}" ixz="${-1.69927e-7 * sim_body_inertia_scale}"/>
     </inertial>
@@ -82,5 +107,5 @@
     <inertial>
       <origin xyz="-0.008867 0.000396 -0.007154" rpy="0 0 0"/>
-      <mass value="0.174884"/>
+      <mass value="${base_link_mass}"/>
       <inertia ixx="${0.00090939 * sim_body_inertia_scale}" iyy="${0.00426716 * sim_body_inertia_scale}" izz="${0.00440707 * sim_body_inertia_scale}" ixy="${1.27324e-7 * sim_body_inertia_scale}" iyz="${1.05509e-9 * sim_body_inertia_scale}" ixz="${-1.69927e-7 * sim_body_inertia_scale}"/>
     </inertial>
@@ -89,5 +114,5 @@
     <inertial>
       <origin xyz="0.020109 0.002332 0.006500" rpy="0 0 0"/>
-      <mass value="${lnkgrp1_weight}"/>
+      <mass value="${lnkgrp1_mass}"/>
       <inertia ixx="${2.494061e-6 * sim_inertia_scale}" iyy="${3.735906e-6 * sim_inertia_scale}" izz="${3.222909e-6 * sim_inertia_scale}" ixy="${-7.662e-9 * sim_inertia_scale}" iyz="${-0.014e-9 * sim_inertia_scale}" ixz="${-33.565e-9 * sim_inertia_scale}"/>
     </inertial>
@@ -109,5 +134,5 @@
     <inertial>
       <origin xyz="-0.003174 0.000986 -0.017984" rpy="0 0 0"/>
-      <mass value="${lnkgrp2_weight}"/>
+      <mass value="${lnkgrp2_mass}"/>
       <inertia ixx="${0.462154e-6 * sim_inertia_scale}" iyy="${0.481174e-6 * sim_inertia_scale}" izz="${26.893e-9 * sim_inertia_scale}" ixy="${3.117e-9 * sim_inertia_scale}" iyz="${17.662e-9 * sim_inertia_scale}" ixz="${-79.269e-9 * sim_inertia_scale}"/>
     </inertial>
@@ -129,5 +154,5 @@
     <inertial>
       <origin xyz="0.006211 0.003456 -0.015014" rpy="0 0 0"/>
-      <mass value="${lnkgrp3_weight}"/>
+      <mass value="${lnkgrp3_mass}"/>
       <inertia ixx="${0.484471e-6 * sim_inertia_scale}" iyy="${0.567615e-6 * sim_inertia_scale}" izz="${91.813e-9 * sim_inertia_scale}" ixy="${-2.101e-9 * sim_inertia_scale}" iyz="${5.008e-9 * sim_inertia_scale}" ixz="${0.20057e-6 * sim_inertia_scale}"/>
     </inertial>
@@ -149,5 +174,5 @@
     <inertial>
       <origin xyz="0.020109 -0.002332 0.006500" rpy="0 0 0"/>
-      <mass value="${lnkgrp1_weight}"/>
+      <mass value="${lnkgrp1_mass}"/>
       <inertia ixx="${2.494061e-06 * sim_inertia_scale}" iyy="${3.735906e-06 * sim_inertia_scale}" izz="${3.222909e-06 * sim_inertia_scale}" ixy="${7.662e-9 * sim_inertia_scale}" iyz="${-0.014e-9 * sim_inertia_scale}" ixz="${-33.565e-9 * sim_inertia_scale}"/>
     </inertial>
@@ -169,5 +194,5 @@
     <inertial>
       <origin xyz="-0.003174 -0.000986 -0.017984" rpy="0 0 0"/>
-      <mass value="${lnkgrp2_weight}"/>
+      <mass value="${lnkgrp2_mass}"/>
       <inertia ixx="${0.462154e-6 * sim_inertia_scale}" iyy="${0.481174e-6 * sim_inertia_scale}" izz="${26.893e-9 * sim_inertia_scale}" ixy="${-3.117e-9 * sim_inertia_scale}" iyz="${-17.662e-9 * sim_inertia_scale}" ixz="${-79.269e-9 * sim_inertia_scale}"/>
     </inertial>
@@ -189,5 +214,5 @@
     <inertial>
       <origin xyz="0.006211 -0.003456 -0.015014" rpy="0 0 0"/>
-      <mass value="${lnkgrp3_weight}"/>
+      <mass value="${lnkgrp3_mass}"/>
       <inertia ixx="${0.484471e-6 * sim_inertia_scale}" iyy="${0.567615e-06 * sim_inertia_scale}" izz="${91.813e-9 * sim_inertia_scale}" ixy="${2.101e-9 * sim_inertia_scale}" iyz="${-5.008e-9 * sim_inertia_scale}" ixz="${0.20057e-6 * sim_inertia_scale}"/>
     </inertial>
@@ -209,5 +234,5 @@
     <inertial>
       <origin xyz="-0.020109 -0.002332 0.006500" rpy="0 0 0"/>
-      <mass value="${lnkgrp1_weight}"/>
+      <mass value="${lnkgrp1_mass}"/>
       <inertia ixx="${2.494061e-06 * sim_inertia_scale}" iyy="${3.735906e-06 * sim_inertia_scale}" izz="${3.222909e-06 * sim_inertia_scale}" ixy="${-7.662e-9 * sim_inertia_scale}" iyz="${-0.014e-9 * sim_inertia_scale}" ixz="${-33.565e-9 * sim_inertia_scale}"/>
     </inertial>
@@ -229,5 +254,5 @@
     <inertial>
       <origin xyz="-0.003174 -0.000986 -0.017984" rpy="0 0 0"/>
-      <mass value="${lnkgrp2_weight}"/>
+      <mass value="${lnkgrp2_mass}"/>
       <inertia ixx="${0.462154e-6 * sim_inertia_scale}" iyy="${0.481174e-6 * sim_inertia_scale}" izz="${26.893e-9 * sim_inertia_scale}" ixy="${-3.117e-9 * sim_inertia_scale}" iyz="${-17.662e-9 * sim_inertia_scale}" ixz="${-79.269e-9 * sim_inertia_scale}"/>
     </inertial>
@@ -249,5 +274,5 @@
     <inertial>
       <origin xyz="0.006211 -0.003456 -0.015014" rpy="0 0 0"/>
-      <mass value="${lnkgrp3_weight}"/>
+      <mass value="${lnkgrp3_mass}"/>
       <inertia ixx="${0.484816e-6 * sim_inertia_scale}" iyy="${0.567883e-06 * sim_inertia_scale}" izz="${91.777e-9 * sim_inertia_scale}" ixy="${2.212e-9 * sim_inertia_scale}" iyz="${-5.34e-9 * sim_inertia_scale}" ixz="${0.200564e-6 * sim_inertia_scale}"/>
     </inertial>
@@ -269,5 +294,5 @@
     <inertial>
       <origin xyz="-0.020109 0.002332 0.006500" rpy="0 0 0"/>
-      <mass value="${lnkgrp1_weight}"/>
+      <mass value="${lnkgrp1_mass}"/>
       <inertia ixx="${2.494061e-06 * sim_inertia_scale}" iyy="${3.735906e-06 * sim_inertia_scale}" izz="${3.222909e-06 * sim_inertia_scale}" ixy="${7.662e-9 * sim_inertia_scale}" iyz="${-0.014e-9 * sim_inertia_scale}" ixz="${-33.565e-9 * sim_inertia_scale}"/>
     </inertial>
@@ -289,5 +314,5 @@
     <inertial>
       <origin xyz="-0.003174 0.000986 -0.017984" rpy="0 0 0"/>
-      <mass value="${lnkgrp2_weight}"/>
+      <mass value="${lnkgrp2_mass}"/>
       <inertia ixx="${0.462154e-6 * sim_inertia_scale}" iyy="${0.481174e-6 * sim_inertia_scale}" izz="${26.893e-9 * sim_inertia_scale}" ixy="${3.117e-9 * sim_inertia_scale}" iyz="${17.662e-9 * sim_inertia_scale}" ixz="${-79.269e-9 * sim_inertia_scale}"/>
     </inertial>
@@ -309,5 +334,5 @@
     <inertial>
       <origin xyz="0.006211 0.003456 -0.015014" rpy="0 0 0"/>
-      <mass value="${lnkgrp3_weight}"/>
+      <mass value="${lnkgrp3_mass}"/>
       <inertia ixx="${0.484471e-6 * sim_inertia_scale}" iyy="${0.567615e-06 * sim_inertia_scale}" izz="${91.813e-9 * sim_inertia_scale}" ixy="${-2.101e-9 * sim_inertia_scale}" iyz="${5.008e-9 * sim_inertia_scale}" ixz="${0.20057e-6 * sim_inertia_scale}"/>
     </inertial>
@@ -329,5 +354,5 @@
     <inertial>
       <origin xyz="-0.005539 -0.000204 0.020223" rpy="0 0 0"/>
-      <mass value="0.00785515871148119"/>
+      <mass value="${body_front_mass}"/>
       <inertia ixx="${5.306048e-6 * sim_body_inertia_scale}" iyy="${1.837621e-6 * sim_body_inertia_scale}" izz="${3.61974e-6 * sim_body_inertia_scale}" ixy="${-22.863e-9 * sim_body_inertia_scale}" iyz="${-4.925e-9 * sim_body_inertia_scale}" ixz="${-9.195e-9 * sim_body_inertia_scale}"/>
     </inertial>
@@ -349,5 +374,5 @@
     <inertial>
       <origin xyz="0.089461 0.023505 0.0" rpy="0 0 0"/>
-      <mass value="0.014261552601793053"/>
+      <mass value="${board_pcb_mass}"/>
       <inertia ixx="${4.425965e-6 * sim_body_inertia_scale}" iyy="${3.4560775e-5 * sim_body_inertia_scale}" izz="${3.8954441e-5 * sim_body_inertia_scale}" ixy="${0.104871e-6 * sim_body_inertia_scale}" iyz="${75.406e-9 * sim_body_inertia_scale}" ixz="${0.113313e-6 * sim_body_inertia_scale}"/>
     </inertial>
@@ -402,5 +427,5 @@
         xyz="1.56706411611127E-05 -5.16565672073303E-13 -0.0191835739440227"
         rpy="0 0 -1.57" />
-      <mass value="0.108" />
+      <mass value="${lidar_mass}" />
       <inertia
         ixx="${8.74731426973985E-06 * sim_body_inertia_scale}"
@@ -432,5 +457,5 @@
     <inertial>
       <origin xyz="${feet_centre_of_mass}" rpy="0 0 0"/>
-      <mass value="${feet_weight}"/>
+      <mass value="${feet_mass}"/>
       <inertia ixx="${41.995e-9 * sim_inertia_scale}" iyy="${62.40e-9 * sim_inertia_scale}" izz="${29.798e-9 * sim_inertia_scale}" ixy="${0.0e-9 * sim_inertia_scale}" iyz="${0.0e-9 * sim_inertia_scale}" ixz="${1.616e-9 * sim_inertia_scale}"/>
     </inertial>
@@ -464,5 +489,5 @@
     <inertial>
       <origin xyz="${feet_centre_of_mass}" rpy="0 0 0"/>
-      <mass value="${feet_weight}"/>
+      <mass value="${feet_mass}"/>
       <inertia ixx="${41.995e-9 * sim_inertia_scale}" iyy="${62.40e-9 * sim_inertia_scale}" izz="${29.798e-9 * sim_inertia_scale}" ixy="${0.0e-9 * sim_inertia_scale}" iyz="${0.0e-9 * sim_inertia_scale}" ixz="${1.616e-9 * sim_inertia_scale}"/>
     </inertial>
@@ -496,5 +521,5 @@
     <inertial>
       <origin xyz="${feet_centre_of_mass}" rpy="0 0 0"/>
-      <mass value="${feet_weight}"/>
+      <mass value="${feet_mass}"/>
       <inertia ixx="${41.995e-9 * sim_inertia_scale}" iyy="${62.40e-9 * sim_inertia_scale}" izz="${29.798e-9 * sim_inertia_scale}" ixy="${0.0e-9 * sim_inertia_scale}" iyz="${0.0e-9 * sim_inertia_scale}" ixz="${1.616e-9 * sim_inertia_scale}"/>
     </inertial>
@@ -528,5 +553,5 @@
     <inertial>
       <origin xyz="${feet_centre_of_mass}" rpy="0 0 0"/>
-      <mass value="${feet_weight}"/>
+      <mass value="${feet_mass}"/>
       <inertia ixx="${41.995e-9 * sim_inertia_scale}" iyy="${62.40e-9 * sim_inertia_scale}" izz="${29.798e-9 * sim_inertia_scale}" ixy="${0.0e-9 * sim_inertia_scale}" iyz="${0.0e-9 * sim_inertia_scale}" ixz="${1.616e-9 * sim_inertia_scale}"/>
     </inertial>
@@ -560,5 +585,5 @@
     <inertial>
       <origin xyz="0.002259 0.008667 -0.002748" rpy="0 0 0"/>
-      <mass value="${pltgrp1_weight}"/>
+      <mass value="${pltgrp1_mass}"/>
       <inertia ixx="${0.39059e-6 * sim_inertia_scale}" iyy="${0.412444e-6 * sim_inertia_scale}" izz="${0.246337e-6 * sim_inertia_scale}" ixy="${24.631e-9 * sim_inertia_scale}" iyz="${3.861e-9 * sim_inertia_scale}" ixz="${54.116e-9 * sim_inertia_scale}"/>
     </inertial>
@@ -580,5 +605,5 @@
     <inertial>
       <origin xyz="0.002259 0.008667 -0.002748" rpy="0 0 0"/>
-      <mass value="${pltgrp1_weight}"/>
+      <mass value="${pltgrp1_mass}"/>
       <inertia ixx="${0.39059e-6 * sim_inertia_scale}" iyy="${0.412444e-6 * sim_inertia_scale}" izz="${0.246337e-6 * sim_inertia_scale}" ixy="${24.631e-9 * sim_inertia_scale}" iyz="${3.861e-9 * sim_inertia_scale}" ixz="${54.116e-9 * sim_inertia_scale}"/>
     </inertial>
@@ -600,5 +625,5 @@
     <inertial>
       <origin xyz="0.002259 -0.008667 -0.002748" rpy="0 0 0"/>
-      <mass value="${pltgrp1_weight}"/>
+      <mass value="${pltgrp1_mass}"/>
       <inertia ixx="${0.39059e-6 * sim_inertia_scale}" iyy="${0.412444e-6 * sim_inertia_scale}" izz="${0.246337e-6 * sim_inertia_scale}" ixy="${-24.631e-9 * sim_inertia_scale}" iyz="${-3.861e-9 * sim_inertia_scale}" ixz="${54.116e-9 * sim_inertia_scale}"/>
     </inertial>
@@ -620,5 +645,5 @@
     <inertial>
       <origin xyz="0.002259 -0.008667 -0.002748" rpy="0 0 0"/>
-      <mass value="${pltgrp1_weight}"/>
+      <mass value="${pltgrp1_mass}"/>
       <inertia ixx="${0.39059e-6 * sim_inertia_scale}" iyy="${0.412444e-6 * sim_inertia_scale}" izz="${0.246337e-6 * sim_inertia_scale}" ixy="${-24.631e-9 * sim_inertia_scale}" iyz="${-3.861e-9 * sim_inertia_scale}" ixz="${54.116e-9 * sim_inertia_scale}"/>
     </inertial>
@@ -640,5 +665,5 @@
     <inertial>
       <origin xyz="-0.001747 0.007904 0.005365" rpy="0 0 0"/>
-      <mass value="${pltgrp2_weight}"/>
+      <mass value="${pltgrp2_mass}"/>
       <inertia ixx="${0.862567e-6 * sim_inertia_scale}" iyy="${0.991403e-6 * sim_inertia_scale}" izz="${0.13904e-6 * sim_inertia_scale}" ixy="${1.254e-9 * sim_inertia_scale}" iyz="${-13.212e-9 * sim_inertia_scale}" ixz="${-0.112894e-6 * sim_inertia_scale}"/>
     </inertial>
@@ -660,5 +685,5 @@
     <inertial>
       <origin xyz="-0.001747 0.007904 0.005365" rpy="0 0 0"/>
-      <mass value="${pltgrp2_weight}"/>
+      <mass value="${pltgrp2_mass}"/>
       <inertia ixx="${0.862567e-6 * sim_inertia_scale}" iyy="${0.991403e-6 * sim_inertia_scale}" izz="${0.13904e-6 * sim_inertia_scale}" ixy="${1.254e-9 * sim_inertia_scale}" iyz="${-13.212e-9 * sim_inertia_scale}" ixz="${-0.112894e-6 * sim_inertia_scale}"/>
     </inertial>
@@ -680,5 +705,5 @@
     <inertial>
       <origin xyz="-0.001747 -0.007904 0.005365" rpy="0 0 0"/>
-      <mass value="${pltgrp2_weight}"/>
+      <mass value="${pltgrp2_mass}"/>
       <inertia ixx="${0.862567e-6 * sim_inertia_scale}" iyy="${0.991403e-6 * sim_inertia_scale}" izz="${0.13904e-6 * sim_inertia_scale}" ixy="${-1.254e-9 * sim_inertia_scale}" iyz="${13.212e-9 * sim_inertia_scale}" ixz="${-0.11152e-6 * sim_inertia_scale}"/>
     </inertial>
@@ -700,5 +725,5 @@
     <inertial>
       <origin xyz="-0.001747 -0.007904 0.005365" rpy="0 0 0"/>
-      <mass value="${pltgrp2_weight}"/>
+      <mass value="${pltgrp2_mass}"/>
       <inertia ixx="${0.862567e-6 * sim_inertia_scale}" iyy="${0.991403e-6 * sim_inertia_scale}" izz="${0.13904e-6 * sim_inertia_scale}" ixy="${-1.254e-9 * sim_inertia_scale}" iyz="${13.212e-9 * sim_inertia_scale}" ixz="${-0.11152e-6 * sim_inertia_scale}"/>
     </inertial>
@@ -720,5 +745,5 @@
     <inertial>
       <origin xyz="-0.00003 0.030005 0.022371" rpy="0 0 0"/>
-      <mass value="0.0051928835390001775"/>
+      <mass value="${shell_side_mass}"/>
       <inertia ixx="${5.834352e-6 * sim_body_inertia_scale}" iyy="${3.214872e-6 * sim_body_inertia_scale}" izz="${6.996514e-6 * sim_body_inertia_scale}" ixy="${0.0e-9 * sim_body_inertia_scale}" iyz="${0.0e-9 * sim_body_inertia_scale}" ixz="${15.218e-9 * sim_body_inertia_scale}"/>
     </inertial>
@@ -1113,5 +1138,5 @@
   <link name="imu_link">
     <inertial>
-      <mass value="0.0001"/>
+      <mass value="${imu_mass}"/>
       <origin rpy="0 0 0" xyz="0 0 0"/>
       <inertia ixx="${1e-09 * sim_body_inertia_scale}" ixy="${0.0 * sim_body_inertia_scale}" ixz="${0.0 * sim_body_inertia_scale}" iyy="${1e-09 * sim_body_inertia_scale}" iyz="${0.0 * sim_body_inertia_scale}" izz="${1e-09 * sim_body_inertia_scale}"/>
