Commit message: Fix the sensors, Change the odom frame for odom in gazebo to

File: mini_pupper_description/urdf/mini_pupper_2/mini_pupper_description.urdf.xacro (robot description, xacro)
@@ -1104,5 +1104,4 @@
     <material>Gazebo/FlatBlack</material>
   </gazebo>
-  <!-- Simplified LIDAR sensor for Gazebo Harmony -->
   <gazebo reference="lidar_link">
     <material>Gazebo/FlatBlack</material>
@@ -1110,8 +1109,7 @@
       <always_on>true</always_on>
       <update_rate>30</update_rate>
-      <topic>/scan</topic>
+      <pose>0 0 0 0 0 0</pose>
       <visualize>false</visualize>
-      <pose>0 0 0 0 0 0</pose>
-      <ray>
+      <lidar>
         <scan>
           <horizontal>
@@ -1119,5 +1117,5 @@
             <resolution>1</resolution>
             <min_angle>0</min_angle>
-            <max_angle>6.283185307179586</max_angle>
+            <max_angle>6.28</max_angle>
           </horizontal>
         </scan>
@@ -1132,13 +1130,22 @@
           <stddev>0.004</stddev>
         </noise>
-      </ray>
+      </lidar>
+      <topic>/scan</topic>
+      <gz_frame_id>lidar_link</gz_frame_id>
     </sensor>
   </gazebo>
-  <!-- Simplified IMU sensor for Gazebo Harmony -->
+  <gazebo>
+    <plugin filename="gz-sim-odometry-publisher-system" name="gz::sim::systems::OdometryPublisher">
+      <odom_frame>odom</odom_frame>
+      <robot_base_frame>base_link</robot_base_frame>
+      <odom_publish_frequency>10.0</odom_publish_frequency>
+      <odom_topic>odom</odom_topic>
+    </plugin>
+  </gazebo>
   <link name="imu_link">
     <inertial>
-      <mass value="${imu_mass}"/>
+      <mass value="0.0001"/>
       <origin rpy="0 0 0" xyz="0 0 0"/>
-      <inertia ixx="${1e-09 * sim_body_inertia_scale}" ixy="${0.0 * sim_body_inertia_scale}" ixz="${0.0 * sim_body_inertia_scale}" iyy="${1e-09 * sim_body_inertia_scale}" iyz="${0.0 * sim_body_inertia_scale}" izz="${1e-09 * sim_body_inertia_scale}"/>
+      <inertia ixx="1e-09" ixy="0.0" ixz="0.0" iyy="1e-09" iyz="0.0" izz="1e-09"/>
     </inertial>
   </link>
@@ -1148,19 +1155,18 @@
   </joint>
   <gazebo reference="imu_link">
-    <sensor name="imu_sensor" type="imu">
+    <sensor name="imu_controller" type="imu">
       <always_on>true</always_on>
       <update_rate>50</update_rate>
       <topic>/imu/data</topic>
+      <gz_frame_id>imu_link</gz_frame_id>
     </sensor>
   </gazebo>
-  <!-- Simplified Camera sensor for Gazebo Harmony -->
+  <!-- Simulated camera mounted to the front body -->
   <link name="camera_link">
     <visual>
       <geometry>
-        <box>
-          <size>0.02 0.02 0.02</size>
-        </box>
-      </geometry>
-      <material>
+        <box size="0.02 0.02 0.02"/>
+      </geometry>
+      <material name="blue">
         <ambient>0 0 1 1</ambient>
         <diffuse>0 0 1 1</diffuse>
@@ -1174,10 +1180,9 @@
   </joint>
   <gazebo reference="camera_link">
-    <sensor name="camera" type="camera">
+    <sensor type="camera" name="sim_camera">
       <always_on>true</always_on>
       <update_rate>30.0</update_rate>
-      <topic>/image_raw</topic>
       <visualize>true</visualize>
-      <camera>
+      <camera name="camera">
         <horizontal_fov>1.3962634</horizontal_fov>
         <image>
@@ -1191,4 +1196,6 @@
         </clip>
       </camera>
+      <topic>/image_raw</topic>
+      <gz_frame_id>camera_link</gz_frame_id>
     </sensor>
   </gazebo>
